File: circuits/ecupnm_nucf103rb/ecupnm_nucf103rb.kicad_sch (KiCad schematic)
At the start: 37 parts, among them J2 Conn_01x03_Male, J2 USB_B_Mini, Q1 2N3904, Q2 IRF540N, Q4 IRF540N, U1 NUCLEO-64, U2 AMS1117-5.0, U3 H11L1, U4 FT232RL, U5 4N35, U7 4N35

Commit message: Update PCB
Parts:
- added J?: Conn_01x03_Male, TerminalBlock:TerminalBlock_Altech_AK300-3_P5.00mm, symbol Connector:Conn_01x03_Male
- added J? (x5): Conn_01x02_Male, TerminalBlock:TerminalBlock_Altech_AK300-2_P5.00mm, symbol Connector:Conn_01x02_Male
- renumbered C1 to C4, C5 to C?, C3 to C?, C7 to C?, C4 to C?, C6 to C?, D4 to D?, D3 to D?, H3 to H?, H1 to H?, H2 to H?, H4 to H?, J2 to J4, J2 to J?, Q4 to Q?, Q2 to Q?, Q1 to Q?, R1 to R7, R9 to R?, R10 to R?, R13 to R?, R19 to R?, R6 to R?, R20 to R?, R11 to R?, R15 to R?, R12 to R?, R14 to R?, R21 to R?, R8 to R?, R7 to R?, U2 to U?, U3 to U?, U5 to U?, U7 to U?, U4 to U?
Connections:
- net +12V: now also J?.1 (Pin_1)
- net GND: now also J?.2 (Pin_2), J?.2 (Pin_2), J?.2 (Pin_2), J?.3 (Pin_3)
- net GNDPWR: now also J?.2 (Pin_2)
- net IN_TPS: now also J?.1 (Pin_1)
- net PORT_IGN: now also J?.2 (Pin_2)
- net PORT_INJ: now also J?.1 (Pin_1)
- net PULSER: now also J?.1 (Pin_1), J?.2 (Pin_2)
- net VCC: now also J?.1 (Pin_1)
- net IN_PULSE: now reaches D?.1 (K), Q?.3 (C), U?.2
- net IN_PULSE: now also J?.1 (Pin_1)
Other:
- moved on the sheet: C?, D?, H?, J4, J?, Q?, R?, U?

Commit message: Nucleo64 PCB
Parts:
- removed D?: D, Diode_SMD:D_SMA-SMB_Universal_Handsoldering, symbol Device:D
- removed J? (x2): Conn_01x03_Male, TerminalBlock:TerminalBlock_Altech_AK300-3_P5.00mm, symbol Connector:Conn_01x03_Male
- removed J? (x5): Conn_01x02_Male, TerminalBlock:TerminalBlock_Altech_AK300-2_P5.00mm, symbol Connector:Conn_01x02_Male
- removed U?: AMS1117-5.0, Package_TO_SOT_SMD:SOT-223-3_TabPin2, symbol Regulator_Linear:AMS1117-5.0
- added D2: 1N4007, Diode_THT:D_DO-41_SOD81_P10.16mm_Horizontal, symbol Diode:1N4007
- added D3: LED, symbol Device:LED
- added J1, J2, J3, JT2, JT3: Conn_01x02_Pin, symbol Connector:Conn_01x02_Pin
- added J4, JT1: Conn_01x03_Pin, symbol Connector:Conn_01x03_Pin
- added R9: 220, symbol Device:R
- added U3: AMS1117-5.0, Package_TO_SOT_SMD:SOT-223-3_TabPin2, symbol Regulator_Linear:AMS1117-5.0
- renumbered J4 to J5, R7 to R8
Connections:
- net +12V: now also JT2.1 (Pin_1), U3.3 (VI)
- net GND: now also D2.2 (A), J1.2 (Pin_2), J2.2 (Pin_2), J3.2 (Pin_2), J4.3 (Pin_3), JT1.3 (Pin_3), U3.1 (GND)
- net GNDPWR: now also D2.1 (K), JT2.2 (Pin_2)
- net IN_PULSE: now also J3.1 (Pin_1)
- net IN_TPS: now also J1.1 (Pin_1)
- net LED_NOCKP: now also D3.1 (K)
- net PORT_IGN: now also JT3.2 (Pin_2)
- net PORT_INJ: now also JT3.1 (Pin_1)
- net PULSER: now also J2.1 (Pin_1), J4.2 (Pin_2)
- net VCC: now also J4.1 (Pin_1), JT1.1 (Pin_1), U3.2 (VO)
- net VDD: now also R9.1
- net at R?.1: now also JT1.2 (Pin_2)
- new net: D3.2 (A), R9.2
- no-connect marks 18 -> 71
Other:
- moved on the sheet: C?, D?, Q?, R?, U?

Commit message: Nucleo 64
Parts:
- C4: footprint (none) -> Capacitor_SMD:C_1206_3216Metric_Pad1.33x1.80mm_HandSolder
- C? (x4): footprint Capacitor_SMD:C_0805_2012Metric_Pad1.18x1.45mm_HandSolder -> Capacitor_SMD:C_1206_3216Metric_Pad1.33x1.80mm_HandSolder
- D3: footprint (none) -> LED_SMD:LED_1206_3216Metric_Pad1.42x1.75mm_HandSolder
- D?: footprint LED_SMD:LED_0805_2012Metric_Pad1.15x1.40mm_HandSolder -> LED_SMD:LED_1206_3216Metric_Pad1.42x1.75mm_HandSolder
- J1, J2, J3: footprint (none) -> Connector_PinSocket_2.54mm:PinSocket_1x02_P2.54mm_Vertical
- J4: footprint (none) -> Connector_PinSocket_2.54mm:PinSocket_1x03_P2.54mm_Vertical
- J5: footprint (none) -> Connector_USB:USB_Mini-B_Wuerth_65100516121_Horizontal
- JT1: footprint (none) -> TerminalBlock:TerminalBlock_Altech_AK300-3_P5.00mm
- JT2, JT3: footprint (none) -> TerminalBlock:TerminalBlock_Altech_AK300-2_P5.00mm
- R8, R9: footprint (none) -> Resistor_SMD:R_1206_3216Metric_Pad1.30x1.75mm_HandSolder
- R? (x13): footprint Resistor_SMD:R_0805_2012Metric_Pad1.20x1.40mm_HandSolder -> Resistor_SMD:R_1206_3216Metric_Pad1.30x1.75mm_HandSolder
- U1: footprint MODULE -> user:Nucleo-64
Changed lines of the file:
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@@
       (effects (font (size 1.27 1.27)))
     )
-    (property "Footprint" "" (at 139.7 51.1048 0)
+    (property "Footprint" "Capacitor_SMD:C_1206_3216Metric_Pad1.33x1.80mm_HandSolder" (at 139.7 51.1048 0)
       (effects (font (size 1.27 1.27)) hide)
     )
@@
       (effects (font (size 1.27 1.27)) hide)
     )
-    (property "Footprint" "" (at 114.3 119.38 0)
+    (property "Footprint" "Connector_PinSocket_2.54mm:PinSocket_1x02_P2.54mm_Vertical" (at 114.3 119.38 0)
       (effects (font (size 1.27 1.27)) hide)
     )
@@
       (effects (font (size 1.27 1.27)) (justify left))
     )
-    (property "Footprint" "Resistor_SMD:R_0805_2012Metric_Pad1.20x1.40mm_HandSolder" (at 94.742 104.14 90)
+    (property "Footprint" "Resistor_SMD:R_1206_3216Metric_Pad1.30x1.75mm_HandSolder" (at 94.742 104.14 90)
       (effects (font (size 1.27 1.27)) hide)
     )
@@
       (effects (font (size 1.27 1.27)) (justify left))
     )
-    (property "Footprint" "Resistor_SMD:R_0805_2012Metric_Pad1.20x1.40mm_HandSolder" (at 122.682 104.14 90)
+    (property "Footprint" "Resistor_SMD:R_1206_3216Metric_Pad1.30x1.75mm_HandSolder" (at 122.682 104.14 90)
       (effects (font (size 1.27 1.27)) hide)
     )
@@
       (effects (font (size 1.27 1.27)) (justify left))
     )
-    (property "Footprint" "Capacitor_SMD:C_0805_2012Metric_Pad1.18x1.45mm_HandSolder" (at 105.1052 175.26 0)
+    (property "Footprint" "Capacitor_SMD:C_1206_3216Metric_Pad1.33x1.80mm_HandSolder" (at 105.1052 175.26 0)
       (effects (font (size 1.27 1.27)) hide)
     )
@@
       (effects (font (size 1.27 1.27)) hide)
     )
-    (property "Footprint" "" (at 30.48 166.37 0)
+    (property "Footprint" "TerminalBlock:TerminalBlock_Altech_AK300-3_P5.00mm" (at 30.48 166.37 0)
       (effects (font (size 1.27 1.27)) hide)
     )
@@
       (effects (font (size 1.27 1.27)) (justify right))
     )
-    (property "Footprint" "LED_SMD:LED_0805_2012Metric_Pad1.15x1.40mm_HandSolder" (at 88.9 114.3 0)
+    (property "Footprint" "LED_SMD:LED_1206_3216Metric_Pad1.42x1.75mm_HandSolder" (at 88.9 114.3 0)
       (effects (font (size 1.27 1.27)) hide)
     )
@@
       (effects (font (size 1.27 1.27)))
     )
-    (property "Footprint" "Resistor_SMD:R_0805_2012Metric_Pad1.20x1.40mm_HandSolder" (at 166.37 47.498 90)
+    (property "Footprint" "Resistor_SMD:R_1206_3216Metric_Pad1.30x1.75mm_HandSolder" (at 166.37 47.498 90)
       (effects (font (size 1.27 1.27)) hide)
     )
@@
       (effects (font (size 1.27 1.27)) hide)
     )
-    (property "Footprint" "" (at 86.36 162.56 0)
+    (property "Footprint" "TerminalBlock:TerminalBlock_Altech_AK300-2_P5.00mm" (at 86.36 162.56 0)
       (effects (font (size 1.27 1.27)) hide)
     )
@@
       (effects (font (size 1.27 1.27)))
     )
-    (property "Footprint" "Resistor_SMD:R_0805_2012Metric_Pad1.20x1.40mm_HandSolder" (at 223.52 47.498 90)
+    (property "Footprint" "Resistor_SMD:R_1206_3216Metric_Pad1.30x1.75mm_HandSolder" (at 223.52 47.498 90)
       (effects (font (size 1.27 1.27)) hide)
     )
@@
       (effects (font (size 1.27 1.27)) (justify left))
     )
-    (property "Footprint" "Resistor_SMD:R_0805_2012Metric_Pad1.20x1.40mm_HandSolder" (at 74.422 120.65 90)
+    (property "Footprint" "Resistor_SMD:R_1206_3216Metric_Pad1.30x1.75mm_HandSolder" (at 74.422 120.65 90)
       (effects (font (size 1.27 1.27)) hide)
     )
@@
       (effects (font (size 1.27 1.27)))
     )
-    (property "Footprint" "MODULE" (at 113.03 22.86 0)
+    (property "Footprint" "user:Nucleo-64" (at 113.03 22.86 0)
       (effects (font (size 1.27 1.27)) hide)
     )
@@
       (effects (font (size 1.27 1.27)) hide)
     )
-    (property "Footprint" "" (at 114.3 129.54 0)
+    (property "Footprint" "Connector_PinSocket_2.54mm:PinSocket_1x03_P2.54mm_Vertical" (at 114.3 129.54 0)
       (effects (font (size 1.27 1.27)) hide)
     )
@@
       (effects (font (size 1.27 1.27)) (justify left))
     )
-    (property "Footprint" "Capacitor_SMD:C_0805_2012Metric_Pad1.18x1.45mm_HandSolder" (at 48.5648 168.91 0)
+    (property "Footprint" "Capacitor_SMD:C_1206_3216Metric_Pad1.33x1.80mm_HandSolder" (at 48.5648 168.91 0)
       (effects (font (size 1.27 1.27)) hide)
     )
@@
       (effects (font (size 1.27 1.27)) (justify left))
     )
-    (property "Footprint" "Resistor_SMD:R_0805_2012Metric_Pad1.20x1.40mm_HandSolder" (at 245.872 41.91 90)
+    (property "Footprint" "Resistor_SMD:R_1206_3216Metric_Pad1.30x1.75mm_HandSolder" (at 245.872 41.91 90)
       (effects (font (size 1.27 1.27)) hide)
     )
@@
       (effects (font (size 1.27 1.27)))
     )
-    (property "Footprint" "" (at 171.45 97.79 0)
+    (property "Footprint" "Connector_USB:USB_Mini-B_Wuerth_65100516121_Horizontal" (at 171.45 97.79 0)
       (effects (font (size 1.27 1.27)) hide)
     )
@@
       (effects (font (size 1.27 1.27)) hide)
     )
-    (property "Footprint" "" (at 31.75 180.34 0)
+    (property "Footprint" "Connector_PinSocket_2.54mm:PinSocket_1x02_P2.54mm_Vertical" (at 31.75 180.34 0)
       (effects (font (size 1.27 1.27)) hide)
     )
@@
       (effects (font (size 1.27 1.27)))
     )
-    (property "Footprint" "Resistor_SMD:R_0805_2012Metric_Pad1.20x1.40mm_HandSolder" (at 45.72 168.148 90)
+    (property "Footprint" "Resistor_SMD:R_1206_3216Metric_Pad1.30x1.75mm_HandSolder" (at 45.72 168.148 90)
       (effects (font (size 1.27 1.27)) hide)
     )
@@
       (effects (font (size 1.27 1.27)) (justify left))
     )
-    (property "Footprint" "Capacitor_SMD:C_0805_2012Metric_Pad1.18x1.45mm_HandSolder" (at 133.6548 167.64 0)
+    (property "Footprint" "Capacitor_SMD:C_1206_3216Metric_Pad1.33x1.80mm_HandSolder" (at 133.6548 167.64 0)
       (effects (font (size 1.27 1.27)) hide)
     )
@@
       (effects (font (size 1.27 1.27)))
     )
-    (property "Footprint" "" (at 135.89 58.928 90)
+    (property "Footprint" "Resistor_SMD:R_1206_3216Metric_Pad1.30x1.75mm_HandSolder" (at 135.89 58.928 90)
       (effects (font (size 1.27 1.27)) hide)
     )
@@
       (effects (font (size 1.27 1.27)) (justify left))
     )
-    (property "Footprint" "Resistor_SMD:R_0805_2012Metric_Pad1.20x1.40mm_HandSolder" (at 197.612 36.83 90)
+    (property "Footprint" "Resistor_SMD:R_1206_3216Metric_Pad1.30x1.75mm_HandSolder" (at 197.612 36.83 90)
       (effects (font (size 1.27 1.27)) hide)
     )
@@
       (effects (font (size 1.27 1.27)) (justify right))
     )
-    (property "Footprint" "Resistor_SMD:R_0805_2012Metric_Pad1.20x1.40mm_HandSolder" (at 57.658 172.72 90)
+    (property "Footprint" "Resistor_SMD:R_1206_3216Metric_Pad1.30x1.75mm_HandSolder" (at 57.658 172.72 90)
       (effects (font (size 1.27 1.27)) hide)
     )
@@
       (effects (font (size 1.27 1.27)) hide)
     )
-    (property "Footprint" "" (at 220.98 26.67 0)
+    (property "Footprint" "TerminalBlock:TerminalBlock_Altech_AK300-2_P5.00mm" (at 220.98 26.67 0)
       (effects (font (size 1.27 1.27)) hide)
     )
@@
       (effects (font (size 1.27 1.27)) (justify left))
     )
-    (property "Footprint" "Resistor_SMD:R_0805_2012Metric_Pad1.20x1.40mm_HandSolder" (at 188.722 41.91 90)
+    (property "Footprint" "Resistor_SMD:R_1206_3216Metric_Pad1.30x1.75mm_HandSolder" (at 188.722 41.91 90)
       (effects (font (size 1.27 1.27)) hide)
     )
@@
       (effects (font (size 1.27 1.27)) (justify left))
     )
-    (property "Footprint" "" (at 139.192 104.14 90)
+    (property "Footprint" "Resistor_SMD:R_1206_3216Metric_Pad1.30x1.75mm_HandSolder" (at 139.192 104.14 90)
       (effects (font (size 1.27 1.27)) hide)
     )
@@
       (effects (font (size 1.27 1.27)) (justify right))
     )
-    (property "Footprint" "" (at 140.97 111.76 0)
+    (property "Footprint" "LED_SMD:LED_1206_3216Metric_Pad1.42x1.75mm_HandSolder" (at 140.97 111.76 0)
       (effects (font (size 1.27 1.27)) hide)
     )
@@
       (effects (font (size 1.27 1.27)) (justify left))
     )
-    (property "Footprint" "Resistor_SMD:R_0805_2012Metric_Pad1.20x1.40mm_HandSolder" (at 254.762 36.83 90)
+    (property "Footprint" "Resistor_SMD:R_1206_3216Metric_Pad1.30x1.75mm_HandSolder" (at 254.762 36.83 90)
       (effects (font (size 1.27 1.27)) hide)
     )
@@
       (effects (font (size 1.27 1.27)))
     )
-    (property "Footprint" "MODULE" (at 52.07 22.86 0)
+    (property "Footprint" "user:Nucleo-64" (at 52.07 22.86 0)
       (effects (font (size 1.27 1.27)) hide)
     )
@@
       (effects (font (size 1.27 1.27)) (justify left))
     )
-    (property "Footprint" "Resistor_SMD:R_0805_2012Metric_Pad1.20x1.40mm_HandSolder" (at 87.122 104.14 90)
+    (property "Footprint" "Resistor_SMD:R_1206_3216Metric_Pad1.30x1.75mm_HandSolder" (at 87.122 104.14 90)
       (effects (font (size 1.27 1.27)) hide)
     )
@@
       (effects (font (size 1.27 1.27)) (justify left))
     )
-    (property "Footprint" "Resistor_SMD:R_0805_2012Metric_Pad1.20x1.40mm_HandSolder" (at 79.502 134.62 90)
+    (property "Footprint" "Resistor_SMD:R_1206_3216Metric_Pad1.30x1.75mm_HandSolder" (at 79.502 134.62 90)
       (effects (font (size 1.27 1.27)) hide)
     )
@@
       (effects (font (size 1.27 1.27)) hide)
     )
-    (property "Footprint" "" (at 64.77 96.52 0)
+    (property "Footprint" "Connector_PinSocket_2.54mm:PinSocket_1x02_P2.54mm_Vertical" (at 64.77 96.52 0)
       (effects (font (size 1.27 1.27)) hide)
     )
@@
       (effects (font (size 1.27 1.27)) (justify left))
     )
-    (property "Footprint" "Capacitor_SMD:C_0805_2012Metric_Pad1.18x1.45mm_HandSolder" (at 75.2348 130.81 0)
-      (effects (font (size 1.27 1.27)) hide)
-    )
+    (property "Footprint" "Capacitor_SMD:C_1206_3216Metric_Pad1.33x1.80mm_HandSolder" (at 75.2348 130.81 0)
+      (effects (font (size 1.27 1.27)) hide)
+    )

Commit message: ECU Nucleo Based
Parts:
- removed H? (x4): MountingHole, MountingHole:MountingHole_2.5mm_Pad, symbol Mechanical:MountingHole
- C?: footprint Capacitor_SMD:C_1206_3216Metric_Pad1.33x1.80mm_HandSolder -> Capacitor_SMD:CP_Elec_4x5.4
- J1: footprint Connector_PinSocket_2.54mm:PinSocket_1x02_P2.54mm_Vertical -> Connector_PinHeader_2.54mm:PinHeader_1x02_P2.54mm_Vertical
- J2: renamed from J3; footprint Connector_PinSocket_2.54mm:PinSocket_1x02_P2.54mm_Vertical -> Connector_PinHeader_2.54mm:PinHeader_1x02_P2.54mm_Vertical
- J3: renamed from J4; footprint Connector_PinSocket_2.54mm:PinSocket_1x03_P2.54mm_Vertical -> Connector_PinHeader_2.54mm:PinHeader_1x03_P2.54mm_Vertical
- JT2: renamed from J2; footprint Connector_PinSocket_2.54mm:PinSocket_1x02_P2.54mm_Vertical -> TerminalBlock:TerminalBlock_Altech_AK300-2_P5.00mm
- Q? (x2): footprint Package_TO_SOT_THT:TO-220-3_Horizontal_TabUp -> Package_TO_SOT_THT:TO-220-3_Horizontal_TabDown
- renumbered C4 to C5, J5 to J4, JT2 to JT3, JT3 to JT4
Connections:
- net VCC: now also U1.6 (E5V); no longer U1.18 (5V)
Other:
- note removed: "HOES"
- moved on the sheet: C5, C?, D2, D3, D?, J1, J2, J3, J4, JT1, JT2, JT3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

Commit message: Ganti Orientasi PCB ECU
Parts:
- removed D3: LED, LED_SMD:LED_1206_3216Metric_Pad1.42x1.75mm_HandSolder, symbol Device:LED
- removed J1, J2: Conn_01x02_Pin, Connector_PinHeader_2.54mm:PinHeader_1x02_P2.54mm_Vertical, symbol Connector:Conn_01x02_Pin
- removed R9: 220, Resistor_SMD:R_1206_3216Metric_Pad1.30x1.75mm_HandSolder, symbol Device:R
- added H1, H2, H3, H4: MountingHole, MountingHole:MountingHole_2.5mm, symbol Mechanical:MountingHole
- C?: footprint Capacitor_SMD:C_Elec_4x5.4 -> Capacitor_THT:CP_Radial_D7.5mm_P2.50mm
- C?: footprint Capacitor_SMD:CP_Elec_4x5.4 -> Capacitor_THT:CP_Radial_D7.5mm_P2.50mm
- renumbered C5 to C2, J3 to J1, J4 to J2, JT2 to JT1, JT3 to JT2, JT1 to JT3, R8 to R6
Connections:
- net LED_NOCKP: no longer names the net of U1.61 (PA8)
- no-connect marks 71 -> 72
Other:
- note added: "Mount Holes"
- moved on the sheet: J1, JT1

Commit message: Serial OK
Other:
- note added: "Correction: 1. Dont connect any STM32 3V3 a) conflict with FTDI 3V3 b) STM32 cant be programmed 2. Temporarily, connect U5V to VCC 5V 3. If using AMS1117-5V a) disconnect U5V b) MOVE THE NUCLEO JUMPER!!"
Changed lines of the file:
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@@
     (effects (font (size 2 2) bold) (justify left bottom))
+  )
+  (text "Correction:\n1. Dont connect any STM32 3V3\n	a) conflict with FTDI 3V3\n	b) STM32 cant be programmed\n2. Temporarily, connect U5V to VCC 5V\n3. If using AMS1117-5V\n	a) disconnect U5V\n	b) MOVE THE NUCLEO JUMPER!!"
+    (at 109.22 189.23 0)
+    (effects (font (size 1.27 1.27)) (justify left bottom))
   )
   (global_label "RX" (shape input) (at 266.7 101.6 0) (fields_autoplaced)
