File: circuits/ecupnm_nucf103rb/ecupnm_nucf103rb.kicad_sch (KiCad schematic)
At the start: 41 parts, among them J1 Conn_01x03_Pin, J2 USB_B_Mini, U1 NUCLEO-64, U3 AMS1117-5.0

Commit message: PCB Nucleo Notes
Other:
- note added: "Correction: 1. Never Connect FTDI 3V3-OUT a) conflict with STM32 3V3 b) use STM32 3V3 for FTDI VCCIO 2. Temporarily, connect U5V to VCC 5V 3. If using AMS1117-5V a) disconnect U5V b) MOVE THE NUCLEO JUMPER!! 4. CKP Input Terminal use 3-pin"
- note removed: "Correction: 1. Dont connect any STM32 3V3 a) conflict with FTDI 3V3 b) STM32 cant be programmed 2. Temporarily, connect U5V to VCC 5V 3. If using AMS1117-5V a) disconnect U5V b) MOVE THE NUCLEO JUMPER!! 4. CKP Input Terminal use 3-pin"
Changed lines of the file:
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@@
     (effects (font (size 2 2) bold) (justify left bottom))
   )
-  (text "Correction:\n1. Dont connect any STM32 3V3\n	a) conflict with FTDI 3V3\n	b) STM32 cant be programmed\n2. Temporarily, connect U5V to VCC 5V\n3. If using AMS1117-5V\n	a) disconnect U5V\n	b) MOVE THE NUCLEO JUMPER!!\n4. CKP Input Terminal use 3-pin"
+  (text "Correction:\n1. Never Connect FTDI 3V3-OUT\n	a) conflict with STM32 3V3\n	b) use STM32 3V3 for FTDI VCCIO\n2. Temporarily, connect U5V to VCC 5V\n3. If using AMS1117-5V\n	a) disconnect U5V\n	b) MOVE THE NUCLEO JUMPER!!\n4. CKP Input Terminal use 3-pin"
     (at 109.22 193.04 0)
     (effects (font (size 1.27 1.27)) (justify left bottom))

Commit message: Update Hasil Tes
Parts:
- added D3, D4: D, Diode_THT:D_DO-15_P10.16mm_Horizontal, symbol Device:D
Connections:
- net GNDPWR: now also D3.2 (A), D4.2 (A)
- net PORT_IGN: now also D3.1 (K)
- net PORT_INJ: now also D4.1 (K)
Changed lines of the file:
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@@
   (junction (at 144.78 151.13) (diameter 0) (color 0 0 0 0)
   )
+  (junction (at 203.2 53.34) (diameter 0) (color 0 0 0 0)
+  )
   (junction (at 139.7 66.04) (diameter 0) (color 0 0 0 0)
   )
@@
   )
   (junction (at 198.12 66.04) (diameter 0) (color 0 0 0 0)
+  )
+  (junction (at 261.62 53.34) (diameter 0) (color 0 0 0 0)
   )
   (junction (at 241.3 146.05) (diameter 0) (color 0 0 0 0)
@@
     (stroke (width 0) (type default))
   )
+  (wire (pts (xy 261.62 60.96) (xy 261.62 66.04))
+    (stroke (width 0) (type default))
+  )
   (wire (pts (xy 44.45 138.43) (xy 44.45 142.24))
     (stroke (width 0) (type default))
@@
     (stroke (width 0) (type default))
   )
+  (wire (pts (xy 203.2 60.96) (xy 203.2 66.04))
+    (stroke (width 0) (type default))
+  )
   (wire (pts (xy 203.2 120.65) (xy 205.74 120.65))
     (stroke (width 0) (type default))
@@
     (stroke (width 0) (type default))
   )
+  (wire (pts (xy 261.62 66.04) (xy 255.27 66.04))
+    (stroke (width 0) (type default))
+  )
   (wire (pts (xy 255.27 41.91) (xy 255.27 44.45))
     (stroke (width 0) (type default))
@@
     (stroke (width 0) (type default))
   )
+  (wire (pts (xy 203.2 66.04) (xy 198.12 66.04))
+    (stroke (width 0) (type default))
+  )
   (wire (pts (xy 87.63 119.38) (xy 87.63 121.92))
     (stroke (width 0) (type default))
@@
     (stroke (width 0) (type default))
   )
+  (wire (pts (xy 261.62 53.34) (xy 267.97 53.34))
+    (stroke (width 0) (type default))
+  )
   (wire (pts (xy 241.3 144.78) (xy 241.3 146.05))
     (stroke (width 0) (type default))
@@
     (stroke (width 0) (type default))
   )
-  (wire (pts (xy 198.12 53.34) (xy 200.66 53.34))
+  (wire (pts (xy 255.27 53.34) (xy 261.62 53.34))
+    (stroke (width 0) (type default))
+  )
+  (wire (pts (xy 198.12 53.34) (xy 203.2 53.34))
     (stroke (width 0) (type default))
   )
@@
     (stroke (width 0) (type default))
   )
+  (wire (pts (xy 203.2 53.34) (xy 210.82 53.34))
+    (stroke (width 0) (type default))
+  )
   (wire (pts (xy 151.13 151.13) (xy 153.67 151.13))
     (stroke (width 0) (type default))
@@
   )
   (wire (pts (xy 168.91 57.15) (xy 171.45 57.15))
-    (stroke (width 0) (type default))
-  )
-  (wire (pts (xy 255.27 53.34) (xy 257.81 53.34))
     (stroke (width 0) (type default))
   )
@@
     (fill (type none))
   )
-  (rectangle (start 154.94 31.75) (end 271.78 76.2)
+  (rectangle (start 154.94 31.75) (end 273.05 76.2)
     (stroke (width 0.1) (type dash))
     (fill (type none))
@@
     )
   )
-  (global_label "PORT_INJ" (shape input) (at 200.66 53.34 0) (fields_autoplaced)
+  (global_label "PORT_INJ" (shape input) (at 210.82 53.34 90) (fields_autoplaced)
     (effects (font (size 1.27 1.27)) (justify left))
-    (property "Intersheetrefs" "${INTERSHEET_REFS}" (at 212.2744 53.34 0)
+    (property "Intersheetrefs" "${INTERSHEET_REFS}" (at 210.82 41.7256 90)
       (effects (font (size 1.27 1.27)) (justify left) hide)
     )
@@
     )
   )
-  (global_label "PORT_IGN" (shape input) (at 257.81 53.34 0) (fields_autoplaced)
+  (global_label "PORT_IGN" (shape input) (at 267.97 53.34 90) (fields_autoplaced)
     (effects (font (size 1.27 1.27)) (justify left))
-    (property "Intersheetrefs" "${INTERSHEET_REFS}" (at 269.7268 53.34 0)
+    (property "Intersheetrefs" "${INTERSHEET_REFS}" (at 267.97 41.4232 90)
       (effects (font (size 1.27 1.27)) (justify left) hide)
     )
@@
   )
   (symbol (lib_id "Transistor_FET:IRF540N") (at 252.73 59.69 0) (unit 1)
-    (in_bom yes) (on_board yes) (dnp no) (fields_autoplaced)
-    (property "Reference" "Q?" (at 259.08 58.4199 0)
-      (effects (font (size 1.27 1.27)) (justify left))
-    )
-    (property "Value" "IRF540N" (at 259.08 60.9599 0)
+    (in_bom yes) (on_board yes) (dnp no)
+    (property "Reference" "Q?" (at 256.54 55.88 0)
+      (effects (font (size 1.27 1.27)) (justify left))
+    )
+    (property "Value" "IRF540N" (at 245.11 64.77 0)
       (effects (font (size 1.27 1.27)) (justify left))
     )
@@
   (symbol (lib_id "Transistor_FET:IRF540N") (at 195.58 59.69 0) (unit 1)
     (in_bom yes) (on_board yes) (dnp no)
-    (property "Reference" "Q?" (at 201.93 58.4199 0)
-      (effects (font (size 1.27 1.27)) (justify left))
-    )
-    (property "Value" "IRF540N" (at 200.66 62.23 0)
+    (property "Reference" "Q?" (at 199.39 55.88 0)
+      (effects (font (size 1.27 1.27)) (justify left))
+    )
+    (property "Value" "IRF540N" (at 187.96 64.77 0)
       (effects (font (size 1.27 1.27)) (justify left))
     )
@@
         )
       )
+    )
+  )
+  (symbol (lib_id "Device:D") (at 261.62 57.15 270) (unit 1)
+    (in_bom yes) (on_board yes) (dnp no) (fields_autoplaced)
+    (property "Reference" "D3" (at 264.16 56.515 90)
+      (effects (font (size 1.27 1.27)) (justify left))
+    )
+    (property "Value" "D" (at 264.16 59.055 90)
+      (effects (font (size 1.27 1.27)) (justify left))
+    )
+    (property "Footprint" "Diode_THT:D_DO-15_P10.16mm_Horizontal" (at 261.62 57.15 0)
+      (effects (font (size 1.27 1.27)) hide)
+    )
+    (property "Datasheet" "~" (at 261.62 57.15 0)
+      (effects (font (size 1.27 1.27)) hide)
+    )
+    (property "Sim.Device" "D" (at 261.62 57.15 0)
+      (effects (font (size 1.27 1.27)) hide)
+    )
+    (property "Sim.Pins" "1=K 2=A" (at 261.62 57.15 0)
+      (effects (font (size 1.27 1.27)) hide)
+    )
+    (pin "1")
+    (pin "2")
+    (instances
+      (project "ecupnm_nucf103rb"
+        (path "/a95c40d2-28a2-42a3-a80e-cd56e62e49d6"
+          (reference "D3") (unit 1)
+        )
+      )
+    )
+  )
+  (symbol (lib_id "Device:D") (at 203.2 57.15 270) (unit 1)
+    (in_bom yes) (on_board yes) (dnp no) (fields_autoplaced)
+    (property "Reference" "D4" (at 205.74 56.515 90)
+      (effects (font (size 1.27 1.27)) (justify left))
+    )
+    (property "Value" "D" (at 205.74 59.055 90)
+      (effects (font (size 1.27 1.27)) (justify left))
+    )
+    (property "Footprint" "Diode_THT:D_DO-15_P10.16mm_Horizontal" (at 203.2 57.15 0)
+      (effects (font (size 1.27 1.27)) hide)
+    )
+    (property "Datasheet" "~" (at 203.2 57.15 0)
+      (effects (font (size 1.27 1.27)) hide)
+    )
+    (property "Sim.Device" "D" (at 203.2 57.15 0)
+      (effects (font (size 1.27 1.27)) hide)
+    )
+    (property "Sim.Pins" "1=K 2=A" (at 203.2 57.15 0)
+      (effects (font (size 1.27 1.27)) hide)
+    )
+    (pin "1")
+    (pin "2")
+    (instances
+      (project "ecupnm_nucf103rb"
+        (path "/a95c40d2-28a2-42a3-a80e-cd56e62e49d6"
+          (reference "D4") (unit 1)
+        )
+      )
