File: circuits/ecupnm_nucf103rb/ecupnm_nucf103rb.kicad_pcb (KiCad board)
At the start: 2 copper layers, 76 x 66 mm, 40 parts, among them J1 Conn_01x03_Pin, J2 USB_B_Mini, Q1 2N3904, Q2 IRF540N, Q3 IRF540N, U1 NUCLEO-64, U2 H11L1, U3 AMS1117-5.0, U4 4N35, U5 4N35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

Commit message: Update Hasil Tes
Parts:
- added C6: 100uF, Capacitor_THT:CP_Radial_D7.5mm_P2.50mm, F.Cu at (211.3, 108.8)
- added D3: D, Diode_THT:D_DO-15_P10.16mm_Horizontal, B.Cu at (169.2, 65.5)
- added D4: D, Diode_THT:D_DO-15_P10.16mm_Horizontal, B.Cu at (145.9, 68.0)
