File: circuits/ecupnm_f051r8/ecupnm_f051r8.kicad_pcb (KiCad board)
At the start: 2 copper layers, 0 parts

Commit message: PCB Baru
Parts:
- added C1: 100nF, Capacitor_SMD:C_0805_2012Metric_Pad1.18x1.45mm_HandSolder, F.Cu at (141.3, 95.0)
- added C2: 100nF, Capacitor_SMD:C_0805_2012Metric_Pad1.18x1.45mm_HandSolder, F.Cu at (159.9, 84.5)
- added C3: 100nF, Capacitor_SMD:C_0805_2012Metric_Pad1.18x1.45mm_HandSolder, F.Cu at (151.3, 66.1)
- added C4: 4u7, Capacitor_SMD:C_0805_2012Metric_Pad1.18x1.45mm_HandSolder, F.Cu at (157.8, 85.8)
- added C5: 100nF, Capacitor_SMD:C_0805_2012Metric_Pad1.18x1.45mm_HandSolder, F.Cu at (145.7, 77.1)
- added C6: 100nF, Capacitor_SMD:C_0805_2012Metric_Pad1.18x1.45mm_HandSolder, F.Cu at (145.7, 83.5)
- added C7: 100uF, Capacitor_THT:CP_Radial_D4.0mm_P2.00mm, F.Cu at (201.9, 91.3)
- added D1: GREEN, LED_SMD:LED_0805_2012Metric_Pad1.15x1.40mm_HandSolder, F.Cu at (151.7, 96.0)
- added D2: BLUE, LED_SMD:LED_0805_2012Metric_Pad1.15x1.40mm_HandSolder, F.Cu at (152.1, 87.1)
- added D3: RED, LED_SMD:LED_0805_2012Metric_Pad1.15x1.40mm_HandSolder, F.Cu at (172.3, 84.5)
- added D4: D, Diode_THT:D_DO-15_P10.16mm_Horizontal, F.Cu at (172.0, 104.5)
- added D5: D, Diode_THT:D_DO-15_P10.16mm_Horizontal, F.Cu at (198.0, 104.6)
- added D6: 1N4007, Diode_THT:D_DO-41_SOD81_P10.16mm_Horizontal, F.Cu at (203.3, 76.6)
- added H1: MountingHole, MountingHole:MountingHole_2.5mm, F.Cu at (132.0, 65.0)
- added H2: MountingHole, MountingHole:MountingHole_2.5mm, F.Cu at (132.0, 109.0)
- added H3: MountingHole, MountingHole:MountingHole_2.5mm, F.Cu at (204.0, 65.0)
- added H4: MountingHole, MountingHole:MountingHole_2.5mm, F.Cu at (204.0, 109.0)
- added J1: Conn_01x03_Pin, Connector_PinHeader_2.54mm:PinHeader_1x03_P2.54mm_Vertical, F.Cu at (145.1, 102.7)
- added J2: Conn_01x03_Pin, Connector_PinHeader_2.54mm:PinHeader_1x03_P2.54mm_Vertical, F.Cu at (146.0, 69.4)
- added J3: Conn_01x05_Pin, Connector_PinHeader_2.54mm:PinHeader_1x05_P2.54mm_Vertical, F.Cu at (156.3, 64.9)
- added J4: Conn_01x03_Pin, Connector_PinHeader_2.54mm:PinHeader_1x03_P2.54mm_Vertical, F.Cu at (197.5, 71.1)
- added J5: USB_B_Mini, Connector_USB:USB_Mini-B_Wuerth_65100516121_Horizontal, F.Cu at (188.9, 66.9)
- added JT1: Conn_01x02_Pin, TerminalBlock:TerminalBlock_Altech_AK300-2_P5.00mm, F.Cu at (133.3, 97.2)
- added JT2: Conn_01x02_Pin, TerminalBlock:TerminalBlock_Altech_AK300-2_P5.00mm, F.Cu at (177.1, 104.9)
- added JT3: Conn_01x03_Pin, TerminalBlock:TerminalBlock_Altech_AK300-3_P5.00mm, F.Cu at (133.5, 83.6)
- added JT4: Conn_01x02_Pin, TerminalBlock:TerminalBlock_Altech_AK300-2_P5.00mm, F.Cu at (198.2, 81.5)
- added Q1: 2N3904, Package_TO_SOT_THT:TO-92_Inline, F.Cu at (146.6, 94.2)
- added Q2: IRF540N, Package_TO_SOT_THT:TO-220-3_Horizontal_TabDown, F.Cu at (167.6, 108.1)
- added Q3: IRF540N, Package_TO_SOT_THT:TO-220-3_Horizontal_TabDown, F.Cu at (194.9, 108.2)
- added R1: 1k, Resistor_SMD:R_0805_2012Metric_Pad1.20x1.40mm_HandSolder, F.Cu at (142.6, 98.0)
- added R10: DNP, Resistor_SMD:R_0805_2012Metric_Pad1.20x1.40mm_HandSolder, F.Cu at (147.8, 87.0)
- added R11: DNP, Resistor_SMD:R_0805_2012Metric_Pad1.20x1.40mm_HandSolder, F.Cu at (163.4, 80.9)
- added R12: 330, Resistor_SMD:R_0805_2012Metric_Pad1.20x1.40mm_HandSolder, F.Cu at (150.0, 87.0)
- added R13: 330, Resistor_SMD:R_0805_2012Metric_Pad1.20x1.40mm_HandSolder, F.Cu at (172.3, 79.6)
- added R14: 220, Resistor_SMD:R_0805_2012Metric_Pad1.20x1.40mm_HandSolder, F.Cu at (169.3, 92.2)
- added R15: 10K, Resistor_SMD:R_0805_2012Metric_Pad1.20x1.40mm_HandSolder, F.Cu at (165.1, 101.3)
- added R16: 10K, Resistor_SMD:R_0805_2012Metric_Pad1.20x1.40mm_HandSolder, F.Cu at (169.4, 101.3)
- added R17: 220, Resistor_SMD:R_0805_2012Metric_Pad1.20x1.40mm_HandSolder, F.Cu at (196.0, 92.2)
- added R18: 10K, Resistor_SMD:R_0805_2012Metric_Pad1.20x1.40mm_HandSolder, F.Cu at (191.8, 101.2)
- added R19: 10K, Resistor_SMD:R_0805_2012Metric_Pad1.20x1.40mm_HandSolder, F.Cu at (195.7, 101.2)
- added R2: 10k, Resistor_SMD:R_0805_2012Metric_Pad1.20x1.40mm_HandSolder, F.Cu at (143.5, 95.0)
- added R20: 1k, Resistor_SMD:R_0805_2012Metric_Pad1.20x1.40mm_HandSolder, F.Cu at (145.7, 79.3)
- added R21: 1k, Resistor_SMD:R_0805_2012Metric_Pad1.20x1.40mm_HandSolder, F.Cu at (145.7, 81.4)
- added R3: 330, Resistor_SMD:R_0805_2012Metric_Pad1.20x1.40mm_HandSolder, F.Cu at (155.3, 94.8)
- added R4: 330, Resistor_SMD:R_0805_2012Metric_Pad1.20x1.40mm_HandSolder, F.Cu at (155.3, 97.0)
- added R5: DNP, Resistor_SMD:R_0805_2012Metric_Pad1.20x1.40mm_HandSolder, F.Cu at (143.7, 106.5)
- added R6: 0, Resistor_SMD:R_0805_2012Metric_Pad1.20x1.40mm_HandSolder, F.Cu at (146.0, 106.5)
- added R7: 10K, Resistor_SMD:R_0805_2012Metric_Pad1.20x1.40mm_HandSolder, F.Cu at (150.2, 109.3)
- added R8: 10K, Resistor_SMD:R_0805_2012Metric_Pad1.20x1.40mm_HandSolder, F.Cu at (145.7, 74.9)
- added R9: 0, Resistor_SMD:R_0805_2012Metric_Pad1.20x1.40mm_HandSolder, F.Cu at (155.7, 85.8)
- added U1: STM32F051R8Tx, Package_QFP:LQFP-64_10x10mm_P0.5mm, F.Cu at (156.1, 75.0)
- added U2: H11L1, Package_DIP:DIP-6_W7.62mm, F.Cu at (154.3, 99.4)
- added U3: 4N35, Package_DIP:DIP-6_W7.62mm, F.Cu at (166.6, 91.5)
- added U4: FT232RL, Package_SO:SSOP-28_5.3x10.2mm_P0.65mm, F.Cu at (175.7, 68.4)
- added U5: 4N35, Package_DIP:DIP-6_W7.62mm, F.Cu at (193.4, 91.4)
- added U6: AMS1117-5.0, Package_TO_SOT_SMD:SOT-223-3_TabPin2, F.Cu at (186.2, 82.8)
- added U7: AMS1117-3.3, Package_TO_SOT_SMD:SOT-223-3_TabPin2, F.Cu at (177.2, 82.0)
Routing:
- net +3V3: track 0.00 -> 219.1 mm, vias 0 -> 6
- net +5V: track 0.00 -> 188.0 mm, vias 0 -> 1
- net GNDPWR: track 0.00 -> 109.3 mm
- net GND: track 0.00 -> 108.0 mm, vias 0 -> 11
- net +12V: track 0.00 -> 87.7 mm
- net OUT_IGN: track 0.00 -> 44.3 mm
- net NRST: track 0.00 -> 41.7 mm
- net IN_CKP: track 0.00 -> 37.0 mm
- net PORT_IGN: track 0.00 -> 33.6 mm
- net QFN_VDD: track 0.00 -> 29.1 mm
- net QFN_VSS: track 0.00 -> 28.8 mm
- net PORT_INJ: track 0.00 -> 24.4 mm
- net Net-(J5-D-): track 0.00 -> 21.4 mm
- net OUT_INJ: track 0.00 -> 19.7 mm
- net BOOT0: track 0.00 -> 18.1 mm
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- added copper zone on F.Cu, net (none)
- added copper zone on B.Cu, net GND
Other:
- board outline added: 80 x 52 mm
- board text added: "12V"
- board text added: "BOOT0"
- board text added: "IGN"
- board text added: "INJ"
- board text added: "Pulser"
- board text added: "SWD"
- board text added: "TPS"
- board text added: "VUSB"
