File: circuits/ecupnm_f051r8/ecupnm_f051r8.kicad_pcb (KiCad board)
At the start: 2 copper layers, 80 x 52 mm, 57 parts, among them J1 Conn_01x03_Pin, J2 Conn_01x03_Pin, J3 Conn_01x05_Pin, J4 Conn_01x03_Pin, J5 USB_B_Mini, Q1 2N3904, Q2 IRF540N, Q3 IRF540N, U1 STM32F051R8Tx, U2 H11L1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

Commit message: Update PCB
Routing:
- net GND: track 108.0 -> 100.2 mm, vias 11 -> 12

Commit message: update PCB
Other:
- board text added: "DATA"

Commit message: update PCB
Other:
- board text added: "SB0"
- board text added: "SB1"
Changed lines of the file:
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@@
     (property "ki_keywords" "R res resistor")
     (attr smd)
-    (fp_text reference "R19" (at 2.86 -10.23) (layer "F.SilkS")
+    (fp_text reference "R19" (at 3.36 0.17) (layer "F.SilkS")
         (effects (font (size 1 1) (thickness 0.15)))
     )
@@
     (property "ki_keywords" "R res resistor")
     (attr smd)
-    (fp_text reference "R10" (at 3.6 0.1 90) (layer "F.SilkS")
+    (fp_text reference "R10" (at 3.6 0.1 90) (layer "F.SilkS") hide
         (effects (font (size 1 1) (thickness 0.15)))
     )
@@
     (property "ki_keywords" "R res resistor")
     (attr smd)
-    (fp_text reference "R11" (at 0 1.8) (layer "F.SilkS")
+    (fp_text reference "R11" (at 0 1.8) (layer "F.SilkS") hide
         (effects (font (size 1 1) (thickness 0.15)))
     )
@@
     (property "ki_keywords" "cap capacitor")
     (attr smd)
-    (fp_text reference "C2" (at 3.5415 -3.278 90) (layer "F.SilkS")
+    (fp_text reference "C2" (at 0.0625 -1.807 90) (layer "F.SilkS")
         (effects (font (size 1 1) (thickness 0.15)))
     )
@@
     (effects (font (size 1.5 1.5) (thickness 0.3) bold) (justify left bottom))
   )
+  (gr_text "SB0" (at 163.2 79.7) (layer "F.SilkS")
+    (effects (font (size 1 1) (thickness 0.15)) (justify left bottom))
+  )
   (gr_text "INJ" (at 177.9 98.3 90) (layer "F.SilkS")
     (effects (font (size 1.5 1.5) (thickness 0.3) bold) (justify left bottom))
@@
     (effects (font (size 1.5 1.5) (thickness 0.3) bold) (justify left bottom))
   )
+  (gr_text "SB1\n" (at 146.5 88.9 90) (layer "F.SilkS")
+    (effects (font (size 1 1) (thickness 0.15)) (justify left bottom))
+  )
   (gr_text "DATA\n" (at 187.5 74) (layer "F.SilkS")
