File: circuits/ecupnm_f051r8_v2/ecu_v2.kicad_pcb (KiCad board)
At the start: 2 copper layers, 99.1 x 33.5 mm, 60 parts, among them J1 Conn_01x03_Pin, J2 Conn_01x05_Pin, J3 USB_B_Mini, J4 Conn_01x03_Pin, J5 Conn_01x03_Pin, Q1 IRF540N, Q2 IRF540N, Q3 2N3904, U1 4N35, U2 4N35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

Commit message: New ECU PCB
Parts:
- moved U6 6.54 mm to (172.2, 86.0), turned to 180 degrees
- moved C9 2.40 mm to (84.2, 99.1)
- moved R18 2.40 mm to (84.2, 101.2)
- moved R20 2.40 mm to (84.2, 97.0)
- moved J5 2.36 mm to (79.2, 102.5)
- moved D6 2.15 mm to (97.2, 95.1)
- moved R13 2.15 mm to (95.2, 95.0)
- moved U7 0.72 mm to (148.9, 92.3)
- moved J3 0.60 mm to (143.4, 83.9)
- moved JT4 0.43 mm to (89.8, 83.0)
Routing:
- net +3V3: track 57.0 -> 198.6 mm, vias 0 -> 8
- net +5V: track 0.00 -> 135.5 mm, vias 0 -> 2
- net +12V: track 1.97 -> 93.4 mm, vias 0 -> 2
- net GND: track 38.3 -> 84.9 mm, vias 8 -> 13
- net OUT_IGN: track 0.00 -> 46.3 mm
- net GNDPWR: track 44.0 -> 83.0 mm
- net Net-(D6-K): track 0.00 -> 21.1 mm
- net Net-(JT4-Pin_2): track 0.14 -> 18.7 mm
- net PULSER: track 0.00 -> 17.8 mm
- net VBUS: track 0.00 -> 17.5 mm
- net Net-(Q3-B): track 4.22 -> 14.0 mm
- net Net-(J5-Pin_1): track 2.33 -> 10.1 mm
- net IN_CKP: track 23.6 -> 27.8 mm
- net Net-(U5-V3): track 0.00 -> 4.06 mm
- net Net-(D5-A): track 0.00 -> 2.22 mm
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- added copper zone on F.Cu, net (none)
- added copper zone on B.Cu, net GND
