File: circuits/ecupnm_f051r8_v2/ecu_v2.kicad_pcb (KiCad board)
At the start: 2 copper layers, 99.1 x 33.5 mm, 60 parts, among them J1 Conn_01x03_Pin, J2 Conn_01x05_Pin, J3 USB_B_Mini, J4 Conn_01x03_Pin, J5 Conn_01x03_Pin, Q1 IRF540N, Q2 IRF540N, Q3 2N3904, U1 4N35, U2 4N35, U3 STM32F051R8Tx, U4 AMS1117-5.0, U5 CH340C, U6 L7805, U7 AMS1117-3.3, U8 H11L1

Commit message: Update New PCB
Parts:
- removed the R10 at (104.0, 105.0)
- removed the R9 at (106.2, 105.0)
- added JP1: Jumper_2_Open, Jumper:SolderJumper-2_P1.3mm_Open_RoundedPad1.0x1.5mm, F.Cu at (105.1, 105.0)
- added JP2: Jumper_2_Open, Jumper:SolderJumper-2_P1.3mm_Open_RoundedPad1.0x1.5mm, F.Cu at (102.3, 105.0)
- moved R10 26.2 mm to (136.7, 93.5)
- moved D5 21.7 mm to (128.6, 91.0)
- moved JT3 1.15 mm to (89.8, 81.9)
- renumbered JT4 to JT3, JT3 to JT4, R12 to R10, R16 to R11, R17 to R12, R18 to R16, R19 to R17, R20 to R18, R21 to R19, R11 to R9
Routing:
- net QFN_VSS: track 25.9 -> 32.9 mm, vias 2 -> 0
- net +3V3: track 198.6 -> 205.4 mm
- net Net-(D5-A): track 2.22 -> 7.06 mm
- net Net-(JT3-Pin_2): track 18.7 -> 19.7 mm
- net QFN_VDD: track 22.7 -> 23.4 mm
Other:
- board text added: "Build by: Deni Nur Fauzi ST MT Achmadi ST MT"
- board text added: "Custom ECU Prototype"
- board text added: "IGN"
- board text added: "INJ"
