File: circuits/ecupnm_f051r8_v2/ecu_v2.kicad_sch (KiCad schematic)
At the start: 60 parts, among them J1 Conn_01x03_Pin, J2 Conn_01x05_Pin, J3 USB_B_Micro, J4 Conn_01x03_Pin, J5 Conn_01x03_Pin, Q1 IRF540N, Q2 IRF540N, Q3 2N3904, U1 4N35, U2 4N35, U3 STM32F051R8Tx, U4 AMS1117-5.0, U5 CH340C, U6 L7805, U7 AMS1117-3.3, U8 H11L1

Commit message: New PCB
Parts:
- removed J3: USB_B_Micro, symbol Connector:USB_B_Micro
- added J3: USB_B_Mini, Connector_USB:USB_Mini-B_Wuerth_65100516121_Horizontal, symbol Connector:USB_B_Mini
- H1, H2, H3, H4: footprint MountingHole:MountingHole_2.5mm -> MountingHole:MountingHole_2.2mm_M2
- U6: footprint (none) -> Package_TO_SOT_THT:TO-220-3_Vertical
Connections:
- net GND: now also J3.5 (GND), J3.6 (Shield)
- net VBUS: now also J3.1 (VBUS)
- net at U5.6 (UD-): now also J3.2 (D-)
- net at U5.5 (UD+): now also J3.3 (D+)
Other:
- note added: "MOUNTING"
- note removed: "MOUNT HOLES"
- moved on the sheet: C8, C9, D6, J5, JT3, JT4, Q3, R13, R14, R15, R16, R17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

Commit message: Update New PCB
Parts:
- removed R10, R9: DNP, Resistor_SMD:R_0805_2012Metric_Pad1.20x1.40mm_HandSolder, symbol Device:R
- added JP1, JP2: Jumper_2_Open, Jumper:SolderJumper-2_P1.3mm_Open_RoundedPad1.0x1.5mm, symbol Jumper:Jumper_2_Open
- renumbered JT4 to JT3, JT3 to JT4, R12 to R10, R16 to R11, R17 to R12, R18 to R16, R19 to R17, R20 to R18, R21 to R19, R11 to R9
Connections:
- net +3V3: now also JP1.2 (B)
- net GND: now also JP2.2 (B)
- net QFN_VDD: now also JP1.1 (A)
- net QFN_VSS: now also JP2.1 (A)
